Commit message: modified:   description/robot_core.xacro

File: description/robot_core.xacro (robot description, xacro)
@@ -23,5 +23,5 @@
         <visual>
             <geometry>
-            <mesh filename="file://$(find hb_description)/models/holonomic_bot/meshes/roller.stl"/>
+            <mesh filename="file:///home/deepanshu/My_ROS/src/ros_bot/hb_description/models/holonomic_bot/meshes/roller.stl"/>
             </geometry>
             <material name="roller_material">
@@ -31,5 +31,5 @@
         <collision>
             <geometry>
-            <mesh filename="file://$(find hb_description)/models/holonomic_bot/meshes/roller.stl"/>
+            <mesh filename="file:///home/deepanshu/My_ROS/src/ros_bot/hb_description/models/holonomic_bot/meshes/roller.stl"/>
             </geometry>
         </collision>
@@ -51,5 +51,5 @@
         <visual>
             <geometry>
-            <mesh filename="file://$(find hb_description)/models/holonomic_bot/meshes/rim.stl"/>
+            <mesh filename="file:///home/deepanshu/My_ROS/src/ros_bot/hb_description/models/holonomic_bot/meshes/rim.stl"/>
             </geometry>
             <material name="rim_${name}_material">
@@ -59,5 +59,5 @@
         <collision>
             <geometry>
-            <mesh filename="file://$(find hb_description)/models/holonomic_bot/meshes/rim.stl"/>
+            <mesh filename="file:///home/deepanshu/My_ROS/src/ros_bot/hb_description/models/holonomic_bot/meshes/rim.stl"/>
             </geometry>
         </collision>
@@ -91,5 +91,5 @@
             <origin xyz="0 0 0" rpy="0 0 0" />
             <geometry>
-                <mesh filename="file://$(find hb_description)/models/holonomic_bot/meshes/bot.dae"/>
+                <mesh filename="file:///home/deepanshu/My_ROS/src/ros_bot/hb_description/models/holonomic_bot/meshes/bot.dae"/>
             </geometry>
         </visual>
@@ -97,5 +97,5 @@
             <origin xyz="0 0 0.026" rpy="0 0 0" />
             <geometry>
-                <mesh filename="file://$(find hb_description)/models/holonomic_bot/meshes/bot.dae"/>
+                <mesh filename="file:///home/deepanshu/My_ROS/src/ros_bot/hb_description/models/holonomic_bot/meshes/bot.dae"/>
             </geometry>
         </collision>
